File: 0_PCBS_Silla/SensorModuleConector/SensorModuleConector.brd (EAGLE design)
At the start: 29.2 x 40 mm, 11 parts

Commit message: 4 marzo
Routing:
- net MOVE: track 81.2 -> 99.4 mm
- net 5V: track 86.9 -> 89.8 mm
- net GND: track 87.8 -> 90.0 mm
- net DIG1: track 29.5 -> 31.4 mm
- net PWM1: track 12.8 -> 11.4 mm
- net PWM2: track 24.5 -> 25.8 mm
- net PWM4: track 22.1 -> 21.3 mm
