File: 0_PCBS_Silla/EagleMotoresI2CAnalogUni/PCBMotoresv3/PCBMotores.brd (EAGLE design)
At the start: 103.7 x 55.1 mm, 30 parts, among them IC1 MEGA8-AI

Commit message: 11 marzo 2020
Parts:
- removed BT: (no value), pinhead:1X04
- added C6, C7: (no value), rcl:153CLV-0505
- added D1, D2: (no value), diode:DO214BA
- added D3: SFH482, led:SFH482
- added IC2: REG1117, burr-brown:SOT223
- added JP3, JP4: (no value), pinhead:1X02
- added Q2: 2SC3838T146, transistor-small-signal:SC59
- added R13, R14: (no value), resistor:M1206
- moved Q1 158.2 mm to (34.6, 3.36), turned to 180 degrees
- moved SERIAL 156.7 mm to (26.1, 7.47)
- moved JP2 140.7 mm to (81.7, 24.8)
- moved LED1 133.6 mm to (7.92, 34.1)
- moved LED2 133.6 mm to (7.82, 27.6)
- moved LED3 133.6 mm to (7.82, 21.0)
- moved LED4 133.6 mm to (7.82, 14.4)
- moved LED5 133.6 mm to (7.82, 7.70)
- moved JP1 109.6 mm to (46.1, 18.3), turned to 270 degrees
- moved R6 108.8 mm to (14.7, 34.2), turned to 180 degrees
- moved R7 108.3 mm to (14.8, 27.7), turned to 180 degrees
- moved R8 107.9 mm to (14.8, 21.0), turned to 180 degrees
- moved R9 107.7 mm to (14.7, 14.4), turned to 180 degrees
- moved R10 107.2 mm to (14.8, 7.68), turned to 180 degrees
- moved SWITCH 102.3 mm to (25.6, 43.0), turned to 270 degrees
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Connections:
- removed net N$21: U$1.12
- new net 3.3V: C6.+, IC2.2, U$1.12
- new net N$15: D1.C, D2.C, R13.1
- new net N$16: Q2.B, R13.2
- new net N$22: D3.K, Q2.C
- new net N$24: JP3.2, U$1.1
- new net N$25: JP4.1, U$1.2
- new net N$26: R14.1, R3.2, R4.1
- net 5V: now also D3.A, IC2.3; no longer BT.1
- net BAT: now also C7.+, R14.2; no longer R3.2, R4.1
- net GND: now also C6.-, C7.-, IC2.1, Q2.E; no longer BT.2
- net N$18: now also D1.A
- net N$19: now also D2.A
- net N$23: now also JP4.2; no longer U$1.2
- net RX-BT: now also JP3.1; no longer BT.3, U$1.1
- net TX-BT: no longer BT.4
Routing:
- net 5V: track 279.0 -> 100.9 mm, vias 2 -> 1
- net GND: track 282.9 -> 127.8 mm, vias 0 -> 1
- net TX-BT: track 80.3 -> 12.2 mm
- net SW1: track 30.4 -> 74.4 mm
- net RX-BT: track 77.6 -> 40.7 mm
- net ANA_D: track 41.8 -> 10.7 mm
- net RX: track 42.1 -> 72.8 mm
- net ANA_I: track 36.1 -> 8.94 mm
- net 3.3V: track 0.00 -> 25.0 mm
- net N$9: track 0.00 -> 22.1 mm
- net RS: track 56.4 -> 34.4 mm, vias 0 -> 1
- net N$23: track 0.00 -> 21.2 mm
- net N$3: track 0.00 -> 20.8 mm
- net N$8: track 0.00 -> 18.3 mm
- net N$6: track 27.4 -> 9.50 mm
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- removed copper zone on layer 16, net GND
Other:
- board size 103.7 x 55.1 mm -> 100 x 50.3 mm

Commit message: 12 marzo 2020
Parts:
- removed D3: SFH482, led:SFH482
- added LED6: (no value), eagle-ltspice:LED_SML0603
- added R15: (no value), resistor:M1206
- D1, D2: device diode:DO214BA -> diode:DO-214AC
- moved R3 11.9 mm to (73.8, 29.7), turned to 180 degrees
- moved SWITCH 9.00 mm to (25.6, 34.0)
- moved D2 7.75 mm to (74.0, 40.3), turned to 90 degrees
- moved R13 6.28 mm to (70.1, 37.0)
- moved Q2 5.28 mm to (74.9, 34.6), turned to 270 degrees
- moved D1 4.13 mm to (77.5, 40.2), turned to 90 degrees
Connections:
- new net N$21: LED6.A, R15.1
- net 5V: now also R15.2; no longer D3.A
- net N$22: now also LED6.C; no longer D3.K
Routing:
- net GND: track 127.8 -> 270.7 mm, vias 1 -> 2
- net BAT: track 0.00 -> 65.1 mm
- net ANA_D: track 10.7 -> 73.7 mm
- net 5V: track 100.9 -> 152.7 mm
- net ANA_I: track 8.94 -> 52.2 mm
- net N$18: track 0.00 -> 40.8 mm
- net N$19: track 0.00 -> 34.0 mm
- net N$26: track 0.00 -> 19.4 mm
- net SW2: track 82.0 -> 92.3 mm, vias 0 -> 1
- net N$22: track 0.00 -> 8.63 mm
- net N$15: track 0.00 -> 7.54 mm
- net N$21: track 0.00 -> 6.20 mm
- net SW1: track 74.4 -> 69.9 mm
- net N$16: track 0.00 -> 3.67 mm
- added copper zone on layer 1, net GND
- added copper zone on layer 16, net GND

Commit message: 13 marzo 2020
Routing:
- net N$26: track 19.4 -> 15.9 mm
- net 5V: track 152.7 -> 154.1 mm
Changed lines of the file:
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@@
 <wire x1="56.5" y1="22.9" x2="56.5" y2="21.251" width="0.4064" layer="1"/>
 <wire x1="56.5" y1="21.251" x2="56.5704" y2="21.1806" width="0.4064" layer="1"/>
-<wire x1="56.49" y1="32.43" x2="56.49" y2="27.79" width="0.4064" layer="1"/>
-<wire x1="56.49" y1="27.79" x2="55.7" y2="27" width="0.4064" layer="1"/>
-<wire x1="55.7" y1="27" x2="55.7" y2="26.46" width="0.4064" layer="1"/>
-<wire x1="55.7" y1="26.46" x2="55.66" y2="26.42" width="0.4064" layer="1"/>
 <wire x1="65.5" y1="5.43" x2="65.5" y2="12.75" width="0.4064" layer="1"/>
 <wire x1="65.5" y1="12.75" x2="65.62" y2="12.87" width="0.4064" layer="1"/>
-<wire x1="55.7" y1="27" x2="55.6" y2="26.9" width="0.4064" layer="1"/>
-<wire x1="55.6" y1="26.9" x2="54.9" y2="26.9" width="0.4064" layer="1"/>
-<wire x1="54.9" y1="26.9" x2="52.9" y2="28.9" width="0.4064" layer="1"/>
-<wire x1="52.9" y1="28.9" x2="52.9" y2="33.7" width="0.4064" layer="1"/>
-<wire x1="52.9" y1="33.7" x2="54.9" y2="35.7" width="0.4064" layer="1"/>
-<wire x1="54.9" y1="35.7" x2="59.4" y2="35.7" width="0.4064" layer="1"/>
-<wire x1="59.4" y1="35.7" x2="65.3" y2="29.8" width="0.4064" layer="1"/>
-<wire x1="65.3" y1="29.8" x2="65.3" y2="26.44" width="0.4064" layer="1"/>
-<wire x1="65.3" y1="26.44" x2="65.32" y2="26.42" width="0.4064" layer="1"/>
 <wire x1="47.35" y1="15.76" x2="47.35" y2="14.95" width="0.4064" layer="16"/>
 <wire x1="47.35" y1="14.95" x2="45" y2="12.6" width="0.4064" layer="16"/>
@@
 <wire x1="29.7" y1="5" x2="26.2" y2="5" width="0.4064" layer="16"/>
 <wire x1="26.2" y1="5" x2="26.13" y2="4.93" width="0.4064" layer="16"/>
-<wire x1="65.3" y1="26.44" x2="65.3" y2="25.2" width="0.4064" layer="1"/>
-<wire x1="65.3" y1="25.2" x2="66.6" y2="23.9" width="0.4064" layer="1"/>
-<wire x1="66.6" y1="23.9" x2="73.1" y2="23.9" width="0.4064" layer="1"/>
-<wire x1="73.1" y1="23.9" x2="75.2" y2="26" width="0.4064" layer="1"/>
-<wire x1="75.2" y1="26" x2="75.2" y2="29.73" width="0.4064" layer="1"/>
-<wire x1="75.2" y1="29.73" x2="75.19" y2="29.74" width="0.4064" layer="1"/>
 <wire x1="75.19" y1="29.74" x2="75.19" y2="30.3" width="0.4064" layer="1"/>
 <wire x1="75.19" y1="30.3" x2="75.19" y2="32.12" width="0.4064" layer="1"/>
@@
 <polygon width="0.4064" layer="16" isolate="1">
 <vertex x="0.1" y="50.1"/>
-<vertex x="100.6" y="50.2"/>
-<vertex x="100.6" y="-0.6"/>
+<vertex x="100.9" y="50.2"/>
+<vertex x="100.9" y="-0.6"/>
 <vertex x="0.2" y="-0.6"/>
 </polygon>
 <polygon width="0.4064" layer="1" isolate="1">
 <vertex x="0.8" y="50"/>
-<vertex x="100.2" y="49.8"/>
-<vertex x="100.2" y="-0.3"/>
+<vertex x="101.9" y="49.8"/>
+<vertex x="101.9" y="-0.3"/>
 <vertex x="0.7" y="-0.3"/>
 </polygon>
+<wire x1="56.49" y1="32.43" x2="56.49" y2="27.25" width="0.4064" layer="1"/>
+<wire x1="56.49" y1="27.25" x2="55.66" y2="26.42" width="0.4064" layer="1"/>
+<wire x1="65.32" y1="26.42" x2="65.32" y2="30.38" width="0.4064" layer="1"/>
+<wire x1="65.32" y1="30.38" x2="59.6" y2="36.1" width="0.4064" layer="1"/>
+<wire x1="59.6" y1="36.1" x2="54.7" y2="36.1" width="0.4064" layer="1"/>
+<wire x1="54.7" y1="36.1" x2="53.3" y2="34.7" width="0.4064" layer="1"/>
+<wire x1="53.3" y1="34.7" x2="53.3" y2="28.78" width="0.4064" layer="1"/>
+<wire x1="53.3" y1="28.78" x2="55.66" y2="26.42" width="0.4064" layer="1"/>
+<wire x1="65.32" y1="26.42" x2="65.32" y2="25.68" width="0.4064" layer="1"/>
+<wire x1="65.32" y1="25.68" x2="66.8" y2="24.2" width="0.4064" layer="1"/>
+<wire x1="66.8" y1="24.2" x2="73" y2="24.2" width="0.4064" layer="1"/>
+<wire x1="73" y1="24.2" x2="75.3" y2="26.5" width="0.4064" layer="1"/>
+<wire x1="75.3" y1="26.5" x2="75.3" y2="29.63" width="0.4064" layer="1"/>
+<wire x1="75.3" y1="29.63" x2="75.19" y2="29.74" width="0.4064" layer="1"/>
 </signal>
 <signal name="RX">
@@
 <wire x1="36.86" y1="19.6326" x2="36.86" y2="17.66" width="0.4064" layer="1"/>
 <wire x1="36.86" y1="17.66" x2="35.3" y2="16.1" width="0.4064" layer="1"/>
-<wire x1="47.35" y1="20.84" x2="47.35" y2="22.05" width="0.4064" layer="1"/>
-<wire x1="47.35" y1="22.05" x2="46.1" y2="23.3" width="0.4064" layer="1"/>
-<wire x1="46.1" y1="23.3" x2="39.4" y2="23.3" width="0.4064" layer="1"/>
-<wire x1="39.4" y1="23.3" x2="36.9" y2="20.8" width="0.4064" layer="1"/>
-<wire x1="36.9" y1="20.8" x2="36.9" y2="19.6726" width="0.4064" layer="1"/>
-<wire x1="36.9" y1="19.6726" x2="36.86" y2="19.6326" width="0.4064" layer="1"/>
 <wire x1="35.48" y1="23.19" x2="35.48" y2="21.18" width="0.4064" layer="1"/>
 <wire x1="35.48" y1="21.18" x2="35.3" y2="21" width="0.4064" layer="1"/>
@@
 <wire x1="83.3" y1="31.2" x2="81.76" y2="31.2" width="0.4064" layer="1"/>
 <wire x1="81.76" y1="31.2" x2="81.73" y2="31.17" width="0.4064" layer="1"/>
+<wire x1="36.86" y1="19.6326" x2="36.86" y2="21.96" width="0.4064" layer="1"/>
+<wire x1="36.86" y1="21.96" x2="38.6" y2="23.7" width="0.4064" layer="1"/>
+<wire x1="38.6" y1="23.7" x2="46.2" y2="23.7" width="0.4064" layer="1"/>
+<wire x1="46.2" y1="23.7" x2="47.4" y2="22.5" width="0.4064" layer="1"/>
+<wire x1="47.4" y1="22.5" x2="47.4" y2="20.89" width="0.4064" layer="1"/>
+<wire x1="47.4" y1="20.89" x2="47.35" y2="20.84" width="0.4064" layer="1"/>
 </signal>
 <signal name="FRENOS">
@@
 <wire x1="63.8" y1="39.2" x2="63.4" y2="39.2" width="0.4064" layer="1"/>
 <wire x1="63.4" y1="39.2" x2="63.23" y2="39.37" width="0.4064" layer="1"/>
-<wire x1="63.23" y1="39.37" x2="63.23" y2="38.37" width="0.4064" layer="1"/>
-<wire x1="63.23" y1="38.37" x2="69.7" y2="31.9" width="0.4064" layer="1"/>
-<wire x1="69.7" y1="31.9" x2="69.7" y2="26.44" width="0.4064" layer="1"/>
-<wire x1="69.7" y1="26.44" x2="69.72" y2="26.42" width="0.4064" layer="1"/>
+<wire x1="63.8" y1="39.2" x2="63.8" y2="34.5" width="0.4064" layer="1"/>
+<wire x1="63.8" y1="34.5" x2="69.6" y2="28.7" width="0.4064" layer="1"/>
+<wire x1="69.6" y1="28.7" x2="69.6" y2="26.54" width="0.4064" layer="1"/>
+<wire x1="69.6" y1="26.54" x2="69.72" y2="26.42" width="0.4064" layer="1"/>
 </signal>
 <signal name="N$10">
@@
 <wire x1="66.03" y1="39.37" x2="66.03" y2="42.56" width="0.4064" layer="1"/>
 <wire x1="66.03" y1="42.56" x2="66.09" y2="42.62" width="0.4064" layer="1"/>
-<wire x1="66.09" y1="42.62" x2="67.18" y2="42.62" width="0.4064" layer="1"/>
-<wire x1="67.18" y1="42.62" x2="68.1" y2="41.7" width="0.4064" layer="1"/>
-<wire x1="68.1" y1="41.7" x2="68.1" y2="34.9" width="0.4064" layer="1"/>
-<wire x1="68.1" y1="34.9" x2="72.4" y2="30.6" width="0.4064" layer="1"/>
-<wire x1="72.4" y1="30.6" x2="72.4" y2="29.75" width="0.4064" layer="1"/>
-<wire x1="72.4" y1="29.75" x2="72.39" y2="29.74" width="0.4064" layer="1"/>
+<wire x1="66.03" y1="39.37" x2="66.03" y2="35.47" width="0.4064" layer="1"/>
+<wire x1="66.03" y1="35.47" x2="71.8" y2="29.7" width="0.4064" layer="1"/>
+<wire x1="71.8" y1="29.7" x2="72.35" y2="29.7" width="0.4064" layer="1"/>
+<wire x1="72.35" y1="29.7" x2="72.39" y2="29.74" width="0.4064" layer="1"/>
 </signal>
 <signal name="N$21">

Commit message: 20 marzo 2020
Parts:
- added R16: (no value), resistor:M1206
- added U$2: PUSH_SMD, push:PUSH_SMD
- moved R3 7.61 mm to (66.9, 32.9)
- moved JP2 6.70 mm to (75.0, 24.9)
- moved D2 5.11 mm to (69.6, 42.9)
- moved D1 5.08 mm to (73.2, 42.9)
- moved Q2 3.10 mm to (74.9, 37.7)
- moved R15 2.87 mm to (82.0, 43.0), turned to 180 degrees
- moved LED6 1.17 mm to (82.6, 40.0)
- moved C7 0.90 mm to (66.6, 26.4)
- moved R13 0.50 mm to (69.6, 37.0)
- renumbered U$1 to BT
Connections:
- net 3.3V: now also U$2.2
- net GND: now also R16.2
- net N$17: now also R16.1, U$2.1
Routing:
- net GND: track 270.6 -> 359.3 mm, vias 2 -> 1
- net 3.3V: track 25.0 -> 63.4 mm
- net N$17: track 0.00 -> 27.6 mm
- net SW2: track 92.3 -> 85.2 mm
- net RX: track 72.8 -> 66.1 mm
- net ANA_I: track 52.2 -> 46.2 mm
- net N$26: track 15.9 -> 9.93 mm
- net SW1: track 69.9 -> 64.1 mm
- net ANA_D: track 73.7 -> 68.0 mm
- net N$19: track 34.0 -> 28.8 mm
- net N$18: track 40.8 -> 35.7 mm
- net N$9: track 22.1 -> 25.8 mm
- net N$21: track 6.20 -> 3.02 mm
- net N$22: track 8.63 -> 6.73 mm
- net N$16: track 3.67 -> 5.39 mm
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Other:
- board size 100 x 50.3 mm -> 95.1 x 50 mm
- board text added: "Control1.0"
- board text added: "INNOVATEC"
