File: 0_PCBS_Silla/EagleMotoresI2CAnalogUni/PCBMotoresv3/PCBMotores.sch (EAGLE design)
At the start: 30 parts, among them IC1 MEGA8-AI

Commit message: 11 marzo 2020
Parts:
- removed BT: (no value), pinhead:PINHD-1X4
- added C6, C7: (no value), rcl:CPOL-EU153CLV-0505
- added D1, D2: (no value), diode:DIODE-DO214BA
- added D3: SFH482, led:SFH482
- added IC2: REG1117, burr-brown:REG1117
- added JP3, JP4: (no value), pinhead:PINHD-1X2
- added Q2: 2SC3838T146, transistor-small-signal:2SC3838T146
- added R13, R14: (no value), resistor:R-EU_M1206
Connections:
- removed net N$21: U$1.3V3
- new net 3.3V: C6.+, IC2.VOUT, U$1.3V3
- new net N$15: D1.C, D2.C, R13.1
- new net N$16: Q2.B, R13.2
- new net N$22: D3.C, Q2.C
- new net N$24: JP3.2, U$1.TX
- new net N$25: JP4.1, U$1.RX
- new net N$26: R14.1, R3.2, R4.1
- net 5V: now also D3.A, IC2.VIN; no longer BT.1
- net BAT: now also C7.+, R14.2; no longer R3.2, R4.1
- net GND: now also C6.-, C7.-, IC2.GND, Q2.E; no longer BT.2
- net N$18: now also D1.A
- net N$19: now also D2.A
- net N$23: now also JP4.2; no longer U$1.RX
- net RX-BT: now also JP3.1; no longer BT.3, U$1.TX
- net TX-BT: no longer BT.4
Other:
- moved on the sheet: R11, R12

Commit message: 12 marzo 2020
Parts:
- removed D3: SFH482, led:SFH482
- added LED6: (no value), eagle-ltspice:LED_ESML0603
- added R15: (no value), resistor:R-EU_M1206
- D1, D2: device diode:DIODE-DO214BA -> diode:DIODE-DO-214AC
Connections:
- new net N$21: LED6.A, R15.1
- net 5V: now also R15.2; no longer D3.A
- net N$22: now also LED6.C; no longer D3.C
Changed lines of the file:
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@@
 <part name="R11" library="resistor" deviceset="R-EU_" device="M1206"/>
 <part name="R12" library="resistor" deviceset="R-EU_" device="M1206"/>
-<part name="D1" library="diode" deviceset="DIODE-" device="DO214BA"/>
-<part name="D2" library="diode" deviceset="DIODE-" device="DO214BA"/>
 <part name="R13" library="resistor" deviceset="R-EU_" device="M1206"/>
 <part name="Q2" library="transistor-small-signal" deviceset="2SC3838" device="T146"/>
-<part name="D3" library="led" deviceset="SFH482" device=""/>
 <part name="C6" library="rcl" deviceset="CPOL-EU" device="153CLV-0505"/>
 <part name="IC2" library="burr-brown" deviceset="REG1117" device=""/>
@@
 <part name="R14" library="resistor" deviceset="R-EU_" device="M1206"/>
 <part name="C7" library="rcl" deviceset="CPOL-EU" device="153CLV-0505"/>
+<part name="LED6" library="eagle-ltspice" deviceset="LED_E" device="SML0603"/>
+<part name="R15" library="resistor" deviceset="R-EU_" device="M1206"/>
+<part name="D1" library="diode" deviceset="DIODE-" device="DO-214AC"/>
+<part name="D2" library="diode" deviceset="DIODE-" device="DO-214AC"/>
 </parts>
 <sheets>
@@
 <instance part="R11" gate="G$1" x="152.4" y="5.08" rot="R90"/>
 <instance part="R12" gate="G$1" x="147.32" y="10.16" rot="R180"/>
-<instance part="D1" gate="G$1" x="228.6" y="7.62"/>
-<instance part="D2" gate="G$1" x="228.6" y="2.54"/>
 <instance part="R13" gate="G$1" x="246.38" y="7.62"/>
 <instance part="Q2" gate="G$1" x="256.54" y="7.62"/>
-<instance part="D3" gate="1" x="259.08" y="25.4"/>
 <instance part="C6" gate="G$1" x="167.64" y="-53.34"/>
 <instance part="IC2" gate="G$1" x="147.32" y="-50.8"/>
@@
 <instance part="R14" gate="G$1" x="175.26" y="50.8" rot="R180"/>
 <instance part="C7" gate="G$1" x="165.1" y="45.72"/>
+<instance part="LED6" gate="G$1" x="259.08" y="25.4"/>
+<instance part="R15" gate="G$1" x="259.08" y="35.56" rot="R90"/>
+<instance part="D1" gate="G$1" x="228.6" y="7.62"/>
+<instance part="D2" gate="G$1" x="228.6" y="2.54"/>
 </instances>
 <busses>
@@
 </segment>
 <segment>
-<pinref part="D3" gate="1" pin="A"/>
-<wire x1="259.08" y1="27.94" x2="259.08" y2="35.56" width="0.1524" layer="91"/>
-<wire x1="259.08" y1="35.56" x2="261.62" y2="35.56" width="0.1524" layer="91"/>
-<label x="264.16" y="35.56" size="1.778" layer="95"/>
-</segment>
-<segment>
 <pinref part="IC2" gate="G$1" pin="VIN"/>
 <wire x1="134.62" y1="-50.8" x2="129.54" y2="-50.8" width="0.1524" layer="91"/>
 <label x="119.38" y="-50.8" size="1.778" layer="95"/>
+</segment>
+<segment>
+<pinref part="R15" gate="G$1" pin="2"/>
+<wire x1="259.08" y1="40.64" x2="259.08" y2="43.18" width="0.1524" layer="91"/>
+<wire x1="259.08" y1="43.18" x2="261.62" y2="43.18" width="0.1524" layer="91"/>
+<label x="264.16" y="43.18" size="1.778" layer="95"/>
 </segment>
 </net>
@@
 <segment>
 <pinref part="U$1" gate="G$1" pin="PIO9"/>
+<wire x1="213.36" y1="7.62" x2="226.06" y2="7.62" width="0.1524" layer="91"/>
 <pinref part="D1" gate="G$1" pin="A"/>
-<wire x1="213.36" y1="7.62" x2="226.06" y2="7.62" width="0.1524" layer="91"/>
 </segment>
 </net>
@@
 <wire x1="213.36" y1="5.08" x2="223.52" y2="5.08" width="0.1524" layer="91"/>
 <wire x1="223.52" y1="5.08" x2="223.52" y2="2.54" width="0.1524" layer="91"/>
+<wire x1="223.52" y1="2.54" x2="226.06" y2="2.54" width="0.1524" layer="91"/>
 <pinref part="D2" gate="G$1" pin="A"/>
-<wire x1="223.52" y1="2.54" x2="226.06" y2="2.54" width="0.1524" layer="91"/>
 </segment>
 </net>
@@
 <net name="N$15" class="0">
 <segment>
-<pinref part="D1" gate="G$1" pin="C"/>
 <wire x1="231.14" y1="7.62" x2="236.22" y2="7.62" width="0.1524" layer="91"/>
 <wire x1="236.22" y1="7.62" x2="236.22" y2="2.54" width="0.1524" layer="91"/>
-<pinref part="D2" gate="G$1" pin="C"/>
 <wire x1="236.22" y1="2.54" x2="231.14" y2="2.54" width="0.1524" layer="91"/>
 <pinref part="R13" gate="G$1" pin="1"/>
 <wire x1="241.3" y1="7.62" x2="236.22" y2="7.62" width="0.1524" layer="91"/>
+<pinref part="D1" gate="G$1" pin="C"/>
+<pinref part="D2" gate="G$1" pin="C"/>
 </segment>
 </net>
@@
 <net name="N$22" class="0">
 <segment>
-<pinref part="D3" gate="1" pin="C"/>
 <pinref part="Q2" gate="G$1" pin="C"/>
 <wire x1="259.08" y1="20.32" x2="259.08" y2="12.7" width="0.1524" layer="91"/>
+<pinref part="LED6" gate="G$1" pin="C"/>
 </segment>
 </net>
@@
 </segment>
 </net>
+<net name="N$21" class="0">
+<segment>
+<pinref part="R15" gate="G$1" pin="1"/>
+<pinref part="LED6" gate="G$1" pin="A"/>
+<wire x1="259.08" y1="30.48" x2="259.08" y2="27.94" width="0.1524" layer="91"/>
+</segment>
+</net>

Commit message: 20 marzo 2020
Parts:
- added R16: (no value), resistor:R-EU_M1206
- added U$2: PUSH_SMD, push:PUSH_SMD
- renumbered U$1 to BT
Connections:
- net 3.3V: now also U$2.2
- net GND: now also R16.2
- net N$17: now also R16.1, U$2.1
Changed lines of the file:
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@@
 <part name="C5" library="rcl" deviceset="C-EU" device="C0402K"/>
 <part name="SWITCH" library="cp150" deviceset="CP150_1X2" device=""/>
-<part name="U$1" library="hc05-own" deviceset="HC-05_BASIC" device=""/>
+<part name="BT" library="hc05-own" deviceset="HC-05_BASIC" device=""/>
 <part name="R11" library="resistor" deviceset="R-EU_" device="M1206"/>
 <part name="R12" library="resistor" deviceset="R-EU_" device="M1206"/>
@@
 <part name="D1" library="diode" deviceset="DIODE-" device="DO-214AC"/>
 <part name="D2" library="diode" deviceset="DIODE-" device="DO-214AC"/>
+<part name="U$2" library="push" deviceset="PUSH_SMD" device=""/>
+<part name="R16" library="resistor" deviceset="R-EU_" device="M1206"/>
 </parts>
 <sheets>
@@
 <instance part="C5" gate="G$1" x="15.24" y="35.56" rot="R180"/>
 <instance part="SWITCH" gate="G$1" x="139.7" y="-5.08" rot="R90"/>
-<instance part="U$1" gate="G$1" x="187.96" y="-2.54"/>
+<instance part="BT" gate="G$1" x="187.96" y="-2.54"/>
 <instance part="R11" gate="G$1" x="152.4" y="5.08" rot="R90"/>
 <instance part="R12" gate="G$1" x="147.32" y="10.16" rot="R180"/>
@@
 <instance part="D1" gate="G$1" x="228.6" y="7.62"/>
 <instance part="D2" gate="G$1" x="228.6" y="2.54"/>
+<instance part="U$2" gate="G$1" x="243.84" y="27.94" rot="R90"/>
+<instance part="R16" gate="G$1" x="223.52" y="22.86" rot="R90"/>
 </instances>
 <busses>
@@
 </segment>
 <segment>
-<pinref part="U$1" gate="G$1" pin="GND"/>
+<pinref part="BT" gate="G$1" pin="GND"/>
 <wire x1="165.1" y1="-17.78" x2="160.02" y2="-17.78" width="0.1524" layer="91"/>
 <label x="152.4" y="-17.78" size="1.778" layer="95"/>
@@
 <wire x1="167.64" y1="-63.5" x2="147.32" y2="-63.5" width="0.1524" layer="91"/>
 <label x="175.26" y="-63.5" size="1.778" layer="95"/>
+</segment>
+<segment>
+<pinref part="R16" gate="G$1" pin="2"/>
+<wire x1="223.52" y1="27.94" x2="223.52" y2="35.56" width="0.1524" layer="91"/>
+<wire x1="223.52" y1="35.56" x2="226.06" y2="35.56" width="0.1524" layer="91"/>
+<label x="226.06" y="35.56" size="1.778" layer="95"/>
 </segment>
 </net>
@@
 </segment>
 </net>
-<net name="N$17" class="0">
-<segment>
-<pinref part="U$1" gate="G$1" pin="PIO11"/>
-<wire x1="213.36" y1="12.7" x2="215.9" y2="12.7" width="0.1524" layer="91"/>
-</segment>
-</net>
 <net name="N$18" class="0">
 <segment>
-<pinref part="U$1" gate="G$1" pin="PIO9"/>
+<pinref part="BT" gate="G$1" pin="PIO9"/>
 <wire x1="213.36" y1="7.62" x2="226.06" y2="7.62" width="0.1524" layer="91"/>
 <pinref part="D1" gate="G$1" pin="A"/>
@@
 <net name="N$19" class="0">
 <segment>
-<pinref part="U$1" gate="G$1" pin="PIO8"/>
+<pinref part="BT" gate="G$1" pin="PIO8"/>
 <wire x1="213.36" y1="5.08" x2="223.52" y2="5.08" width="0.1524" layer="91"/>
 <wire x1="223.52" y1="5.08" x2="223.52" y2="2.54" width="0.1524" layer="91"/>
@@
 <net name="N$20" class="0">
 <segment>
-<pinref part="U$1" gate="G$1" pin="LED"/>
+<pinref part="BT" gate="G$1" pin="LED"/>
 <wire x1="213.36" y1="-17.78" x2="215.9" y2="-17.78" width="0.1524" layer="91"/>
 </segment>
@@
 </segment>
 <segment>
-<pinref part="U$1" gate="G$1" pin="3V3"/>
+<pinref part="BT" gate="G$1" pin="3V3"/>
 <wire x1="165.1" y1="-15.24" x2="160.02" y2="-15.24" width="0.1524" layer="91"/>
 <label x="152.4" y="-15.24" size="1.778" layer="95"/>
 </segment>
+<segment>
+<pinref part="U$2" gate="G$1" pin="2"/>
+<wire x1="236.22" y1="33.02" x2="236.22" y2="38.1" width="0.1524" layer="91"/>
+<wire x1="236.22" y1="38.1" x2="238.76" y2="38.1" width="0.1524" layer="91"/>
+<label x="238.76" y="38.1" size="1.778" layer="95"/>
+</segment>
 </net>
 <net name="N$24" class="0">
 <segment>
-<pinref part="U$1" gate="G$1" pin="TX"/>
+<pinref part="BT" gate="G$1" pin="TX"/>
 <pinref part="JP3" gate="G$1" pin="2"/>
 <wire x1="165.1" y1="12.7" x2="160.02" y2="12.7" width="0.1524" layer="91"/>
@@
 <net name="N$25" class="0">
 <segment>
-<pinref part="U$1" gate="G$1" pin="RX"/>
+<pinref part="BT" gate="G$1" pin="RX"/>
 <pinref part="JP4" gate="G$1" pin="1"/>
 <wire x1="165.1" y1="10.16" x2="162.56" y2="10.16" width="0.1524" layer="91"/>
@@
 </segment>
 </net>
+<net name="N$17" class="0">
+<segment>
+<pinref part="BT" gate="G$1" pin="PIO11"/>
+<pinref part="U$2" gate="G$1" pin="1"/>
+<wire x1="213.36" y1="12.7" x2="223.52" y2="12.7" width="0.1524" layer="91"/>
+<wire x1="223.52" y1="12.7" x2="236.22" y2="12.7" width="0.1524" layer="91"/>
+<wire x1="236.22" y1="12.7" x2="236.22" y2="22.86" width="0.1524" layer="91"/>
+<pinref part="R16" gate="G$1" pin="1"/>
+<wire x1="223.52" y1="17.78" x2="223.52" y2="12.7" width="0.1524" layer="91"/>
+</segment>
+</net>
