File: 0_PCBS_Silla/SensorLaser/SensorLaser.brd (EAGLE design)
At the start: 28.9 x 27.3 mm, 11 parts, among them IC1 MEGA8-AI

Commit message: 20 marzo 2020
Parts:
- moved SENSOR 1.20 mm to (12.6, 23.0)
- moved BUZZ 1.20 mm to (12.6, 6.26)
- moved R1 1.20 mm to (4.78, 19.1)
- moved IC1 1.20 mm to (12.4, 14.5)
- moved U$1 1.20 mm to (21.6, 4.60)
- moved U$2 1.20 mm to (21.4, 12.7)
- moved Q2 1.20 mm to (3.82, 10.8)
- moved DATA 1.20 mm to (12.4, 3.70)
- moved C1 1.00 mm to (5.66, 3.58)
- moved C2 0.86 mm to (7.28, 3.59)
- moved C3 0.71 mm to (19.6, 17.8)
Routing:
- net 5V: track 73.0 -> 76.1 mm
- net N$7: track 15.1 -> 16.0 mm
- net N$6: track 11.1 -> 11.6 mm
Other:
- board size 28.9 x 27.3 mm -> 26 x 25.1 mm
- board text added: "Innovatec"
- board text added: "SL1.0"
