File: 0_PCBS_Silla/SensorLaser/SensorLaser.sch (EAGLE design)
At the start: 11 parts, among them IC1 MEGA8-AI

Commit message: 4 marzo
Connections:
- removed net N$19: BUZZ.+, IC1.PD2(INT0)
- removed net N$20: IC1.PD3(INT1), U$2.1
- new net N$1: BUZZ.+, IC1.PB2(SS/OC1B)
- net MOVE: now also IC1.PD7(AIN1); no longer IC1.PD4(XCK/T0)
- net SCK: now also U$2.1
Changed lines of the file:
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@@
 <setting verticaltext="up"/>
 </settings>
-<grid distance="0.1" unitdist="inch" unit="inch" style="lines" multiple="1" display="yes" altdistance="0.01" altunitdist="inch" altunit="inch"/>
+<grid distance="0.1" unitdist="inch" unit="inch" style="lines" multiple="1" display="no" altdistance="0.01" altunitdist="inch" altunit="inch"/>
 <layers>
 <layer number="1" name="Top" color="4" fill="1" visible="no" active="no"/>
@@
 <instance part="DATA" gate="G$1" x="48.26" y="-5.08" rot="R180"/>
 <instance part="U$1" gate="G$1" x="25.4" y="-35.56"/>
-<instance part="U$2" gate="G$1" x="10.16" y="-17.78"/>
+<instance part="U$2" gate="G$1" x="20.32" y="-20.32"/>
 </instances>
 <busses>
@@
 <pinref part="U$2" gate="G$1" pin="2"/>
 <pinref part="BUZZ" gate="G$1" pin="-"/>
-<wire x1="15.24" y1="-10.16" x2="25.4" y2="-10.16" width="0.1524" layer="91"/>
-<wire x1="25.4" y1="-10.16" x2="25.4" y2="0" width="0.1524" layer="91"/>
+<wire x1="25.4" y1="-12.7" x2="25.4" y2="0" width="0.1524" layer="91"/>
 <wire x1="25.4" y1="0" x2="27.94" y2="0" width="0.1524" layer="91"/>
 <label x="30.48" y="0" size="1.778" layer="95"/>
@@
 <label x="-2.54" y="-30.48" size="1.778" layer="95"/>
 </segment>
+<segment>
+<pinref part="U$2" gate="G$1" pin="1"/>
+<wire x1="15.24" y1="-12.7" x2="12.7" y2="-12.7" width="0.1524" layer="91"/>
+<label x="5.08" y="-12.7" size="1.778" layer="95"/>
+</segment>
 </net>
 <net name="MISO" class="0">
@@
 </segment>
 </net>
-<net name="N$19" class="0">
-<segment>
-<pinref part="IC1" gate="G$1" pin="PD2(INT0)"/>
-<pinref part="BUZZ" gate="G$1" pin="+"/>
-<wire x1="-7.62" y1="0" x2="5.08" y2="0" width="0.1524" layer="91"/>
-</segment>
-</net>
-<net name="N$20" class="0">
-<segment>
-<pinref part="U$2" gate="G$1" pin="1"/>
-<wire x1="5.08" y1="-10.16" x2="5.08" y2="-2.54" width="0.1524" layer="91"/>
-<pinref part="IC1" gate="G$1" pin="PD3(INT1)"/>
-<wire x1="5.08" y1="-2.54" x2="-7.62" y2="-2.54" width="0.1524" layer="91"/>
-</segment>
-</net>
 <net name="MOVE" class="0">
 <segment>
@@
 </segment>
 <segment>
-<pinref part="IC1" gate="G$1" pin="PD4(XCK/T0)"/>
-<wire x1="-7.62" y1="-5.08" x2="-5.08" y2="-5.08" width="0.1524" layer="91"/>
-<label x="-2.54" y="-5.08" size="1.778" layer="95"/>
-</segment>
-</net>
+<pinref part="IC1" gate="G$1" pin="PD7(AIN1)"/>
+<wire x1="-7.62" y1="-12.7" x2="-5.08" y2="-12.7" width="0.1524" layer="91"/>
+<label x="-2.54" y="-12.7" size="1.778" layer="95"/>
+</segment>
+</net>
+<net name="N$1" class="0">
+<segment>
+<pinref part="BUZZ" gate="G$1" pin="+"/>
+<wire x1="5.08" y1="0" x2="2.54" y2="0" width="0.1524" layer="91"/>
+<wire x1="2.54" y1="0" x2="2.54" y2="-22.86" width="0.1524" layer="91"/>
+<pinref part="IC1" gate="G$1" pin="PB2(SS/OC1B)"/>
+<wire x1="2.54" y1="-22.86" x2="-7.62" y2="-22.86" width="0.1524" layer="91"/>
+</segment>
+</net>
