File: 0_PCBS_Silla/SensorModule/SensorModule.brd (EAGLE design)
At the start: 80.1 x 65.5 mm, 32 parts, among them IC1 MEGA8-AI, K1 G5LE, Q2 BC547B, Q3 BC547B

Commit message: 20 marzo 2020
Parts:
- added LED1, LED2: (no value), led:CHIP-LED0603
- added R10, R11, R12: (no value), rcl:M1206
- renumbered CONTACTOR to CONTAC
Connections:
- new net N$5: LED1.C, R10.2
- new net N$8: LED2.A, R11.2
- net 5V: now also LED1.A, R12.2
- net GND: now also LED2.C
- net N$2: now also R10.1, R11.1, R12.1
Routing:
- net 5V: track 185.6 -> 201.7 mm
- net N$2: track 16.9 -> 29.6 mm
- net N$5: track 0.00 -> 10.6 mm
- net GND: track 284.5 -> 293.3 mm
- net N$8: track 0.00 -> 2.44 mm
- net PWM6: track 36.2 -> 35.2 mm
- net ANA_D: track 20.0 -> 20.5 mm
Other:
- board text added: "+"
- board text added: "-"
- board text added: "INNOVATEC"
- board text added: "SENSOR_MODULE_1.0"
