File: 0_PCBS_Silla/SensorModule/SensorModule.sch (EAGLE design)
At the start: 32 parts, among them IC1 MEGA8-AI, K1 G5LE, Q2 BC547B, Q3 BC547B

Commit message: 20 marzo 2020
Parts:
- added LED1, LED2: (no value), led:LEDCHIP-LED0603
- added R10, R11, R12: (no value), rcl:R-EU_M1206
- renumbered CONTACTOR to CONTAC
Connections:
- new net N$5: LED1.C, R10.2
- new net N$8: LED2.A, R11.2
- net 5V: now also LED1.A, R12.2
- net GND: now also LED2.C
- net N$2: now also R10.1, R11.1, R12.1
Changed lines of the file:
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@@
 <part name="JP1" library="pinhead" deviceset="PINHD-1X8" device=""/>
 <part name="D1" library="diode" deviceset="1N4004" device=""/>
-<part name="CONTACTOR" library="con-ptr500" deviceset="AK500/2" device=""/>
+<part name="CONTAC" library="con-ptr500" deviceset="AK500/2" device=""/>
 <part name="Q3" library="transistor-npn" deviceset="BC547*" device="" technology="B"/>
 <part name="R9" library="rcl" deviceset="R-EU_" device="M1206"/>
@@
 <part name="C8" library="rcl" deviceset="CPOL-EU" device="153CLV-0505"/>
 <part name="C9" library="rcl" deviceset="CPOL-EU" device="153CLV-0505"/>
+<part name="R10" library="rcl" deviceset="R-EU_" device="M1206"/>
+<part name="R11" library="rcl" deviceset="R-EU_" device="M1206"/>
+<part name="R12" library="rcl" deviceset="R-EU_" device="M1206"/>
+<part name="LED1" library="led" deviceset="LED" device="CHIP-LED0603"/>
+<part name="LED2" library="led" deviceset="LED" device="CHIP-LED0603"/>
 </parts>
 <sheets>
@@
 <instance part="JP1" gate="A" x="134.62" y="58.42" rot="R180"/>
 <instance part="D1" gate="1" x="60.96" y="86.36"/>
-<instance part="CONTACTOR" gate="-1" x="200.66" y="63.5"/>
-<instance part="CONTACTOR" gate="-2" x="200.66" y="58.42"/>
+<instance part="CONTAC" gate="-1" x="200.66" y="63.5"/>
+<instance part="CONTAC" gate="-2" x="200.66" y="58.42"/>
 <instance part="Q3" gate="G$1" x="17.78" y="53.34"/>
 <instance part="R9" gate="G$1" x="5.08" y="53.34"/>
@@
 <instance part="C8" gate="G$1" x="132.08" y="-15.24" rot="R270"/>
 <instance part="C9" gate="G$1" x="132.08" y="-25.4" rot="R270"/>
+<instance part="R10" gate="G$1" x="27.94" y="86.36" rot="R90"/>
+<instance part="R11" gate="G$1" x="38.1" y="86.36" rot="R90"/>
+<instance part="R12" gate="G$1" x="48.26" y="86.36" rot="R90"/>
+<instance part="LED1" gate="G$1" x="27.94" y="99.06"/>
+<instance part="LED2" gate="G$1" x="38.1" y="96.52" rot="R180"/>
 </instances>
 <busses>
@@
 <wire x1="73.66" y1="0" x2="68.58" y2="0" width="0.1524" layer="91"/>
 <label x="60.96" y="0" size="1.778" layer="95"/>
+</segment>
+<segment>
+<wire x1="27.94" y1="101.6" x2="27.94" y2="106.68" width="0.1524" layer="91"/>
+<wire x1="27.94" y1="106.68" x2="25.4" y2="106.68" width="0.1524" layer="91"/>
+<label x="20.32" y="106.68" size="1.778" layer="95"/>
+<pinref part="LED1" gate="G$1" pin="A"/>
+</segment>
+<segment>
+<pinref part="R12" gate="G$1" pin="2"/>
+<wire x1="48.26" y1="91.44" x2="48.26" y2="96.52" width="0.1524" layer="91"/>
+<wire x1="48.26" y1="96.52" x2="50.8" y2="96.52" width="0.1524" layer="91"/>
+<label x="53.34" y="96.52" size="1.778" layer="95"/>
 </segment>
 </net>
@@
 <label x="60.96" y="-2.54" size="1.778" layer="95"/>
 </segment>
+<segment>
+<wire x1="38.1" y1="101.6" x2="38.1" y2="106.68" width="0.1524" layer="91"/>
+<wire x1="38.1" y1="106.68" x2="40.64" y2="106.68" width="0.1524" layer="91"/>
+<label x="43.18" y="106.68" size="1.778" layer="95"/>
+<pinref part="LED2" gate="G$1" pin="C"/>
+</segment>
 </net>
 <net name="DIG1" class="0">
@@
 <segment>
 <pinref part="Q2" gate="G$1" pin="C"/>
-<wire x1="20.32" y1="76.2" x2="55.88" y2="76.2" width="0.1524" layer="91"/>
+<wire x1="20.32" y1="76.2" x2="27.94" y2="76.2" width="0.1524" layer="91"/>
 <pinref part="K1" gate="1" pin="2"/>
 <pinref part="D1" gate="1" pin="A"/>
+<wire x1="27.94" y1="76.2" x2="38.1" y2="76.2" width="0.1524" layer="91"/>
+<wire x1="38.1" y1="76.2" x2="48.26" y2="76.2" width="0.1524" layer="91"/>
+<wire x1="48.26" y1="76.2" x2="55.88" y2="76.2" width="0.1524" layer="91"/>
 <wire x1="58.42" y1="86.36" x2="55.88" y2="86.36" width="0.1524" layer="91"/>
 <wire x1="55.88" y1="86.36" x2="55.88" y2="76.2" width="0.1524" layer="91"/>
+<pinref part="R10" gate="G$1" pin="1"/>
+<wire x1="27.94" y1="81.28" x2="27.94" y2="76.2" width="0.1524" layer="91"/>
+<pinref part="R11" gate="G$1" pin="1"/>
+<wire x1="38.1" y1="81.28" x2="38.1" y2="76.2" width="0.1524" layer="91"/>
+<pinref part="R12" gate="G$1" pin="1"/>
+<wire x1="48.26" y1="81.28" x2="48.26" y2="76.2" width="0.1524" layer="91"/>
 </segment>
 </net>
@@
 </segment>
 <segment>
-<pinref part="CONTACTOR" gate="-2" pin="KL"/>
+<pinref part="CONTAC" gate="-2" pin="KL"/>
 <wire x1="205.74" y1="58.42" x2="208.28" y2="58.42" width="0.1524" layer="91"/>
 <label x="210.82" y="58.42" size="1.778" layer="95"/>
@@
 </segment>
 <segment>
-<pinref part="CONTACTOR" gate="-1" pin="KL"/>
+<pinref part="CONTAC" gate="-1" pin="KL"/>
 <wire x1="205.74" y1="63.5" x2="208.28" y2="63.5" width="0.1524" layer="91"/>
 <label x="210.82" y="63.5" size="1.778" layer="95"/>
@@
 </segment>
 </net>
+<net name="N$5" class="0">
+<segment>
+<pinref part="R10" gate="G$1" pin="2"/>
+<wire x1="27.94" y1="93.98" x2="27.94" y2="91.44" width="0.1524" layer="91"/>
+<pinref part="LED1" gate="G$1" pin="C"/>
+</segment>
+</net>
+<net name="N$8" class="0">
+<segment>
+<pinref part="R11" gate="G$1" pin="2"/>
+<wire x1="38.1" y1="93.98" x2="38.1" y2="91.44" width="0.1524" layer="91"/>
+<pinref part="LED2" gate="G$1" pin="A"/>
+</segment>
+</net>
